Commit message: Changed inertial origin as the visual one

File: src/turtlebot3/turtlebot3_description/urdf/turtlebot3_waffle.urdf.xacro (robot description, xacro)
@@ -28,5 +28,6 @@
     </collision>
     <inertial>
-      <origin xyz="0 0 0" rpy="0 0 0"/>
+      <!-- Changed inertial origin as the visual one-->
+      <origin xyz="-0.064 0 0" rpy="0 0 0"/>
       <mass value="1.3729096e+00"/>
       <inertia ixx="8.7002718e-03" ixy="-4.7576583e-05" ixz="1.1160499e-04"
@@ -184,5 +185,5 @@
     </collision>
     <!-- This inertial field needs doesn't contain reliable data!! -->
-<!--   <inertial>
+    <inertial>
       <mass value="0.564" />
       <origin xyz="0 0 0" />
@@ -190,5 +191,5 @@
                iyy="0.000498940" iyz="0.0"
                izz="0.003879257" />
-    </inertial>-->
+    </inertial>
   </link>
   <joint name="camera_rgb_joint" type="fixed">
